Commit message: add robots collision

File: data/robots/irb4600/irb4600.urdf (robot description, URDF)
Before this commit: robot irb4600, 7 links, 6 joints
Links:
- link base_link: geometry collision mesh filename=meshes/IRB4600_40kg-255_IRC5_rev04_Base.obj scale=0.001; visual mesh filename=meshes/IRB4600_40kg-255_IRC5_rev04_Base.obj scale=0.001
- link link_1: geometry collision mesh filename=meshes/IRB4600_40kg-255_IRC5_rev04_Link1.obj scale=0.001; visual mesh filename=meshes/IRB4600_40kg-255_IRC5_rev04_Link1.obj scale=0.001
- link link_2: geometry collision mesh filename=meshes/IRB4600_40kg-255_IRC5_rev04_Link2.obj scale=0.001; visual mesh filename=meshes/IRB4600_40kg-255_IRC5_rev04_Link2.obj scale=0.001
- link link_3: geometry collision mesh filename=meshes/IRB4600_40kg-255_IRC5_rev04_Link3.obj scale=0.001; visual mesh filename=meshes/IRB4600_40kg-255_IRC5_rev04_Link3.obj scale=0.001
- link link_4: geometry collision mesh filename=meshes/IRB4600_40kg-255_IRC5_rev04_Link4.obj scale=0.001; visual mesh filename=meshes/IRB4600_40kg-255_IRC5_rev04_Link4.obj scale=0.001
- link link_5: geometry collision mesh filename=meshes/IRB4600_40kg-255_IRC5_rev04_Link5.obj scale=0.001; visual mesh filename=meshes/IRB4600_40kg-255_IRC5_rev04_Link5.obj scale=0.001
- link link_6: geometry collision mesh filename=meshes/IRB4600_40kg-255_IRC5_rev04_Link6.obj scale=0.001; visual mesh filename=meshes/IRB4600_40kg-255_IRC5_rev04_Link6.obj scale=0.001
